File: dryer_adc_8_stm32.kicad_pcb (KiCad board)
At the start: 2 copper layers, 78 x 28 mm, 78 parts, among them J11 SWD, J12 NODE, J13 BOOTLDR, J14 Clamp_Terminal_01x09, J18 B6B, J19 B6B, U11 STM32G070CBTx, U12 74LVC1G07, U13 HXY6206I-3V3, U14 74LVC1G07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

Commit message: ready to production
Routing:
- net ENSPWR: track 55.6 -> 54.9 mm, vias 3 -> 2
- net SWDIO: track 34.9 -> 34.3 mm
