File: dryer_adc_8_stm32.kicad_sch (KiCad schematic)
At the start: 78 parts, among them J11 SWD, J12 NODE, J13 BOOTLDR, J14 Clamp_Terminal_01x09, J18 B6B, J19 B6B, U11 STM32G070CBTx, U12 74LVC1G07, U13 HXY6206I-3V3, U14 74LVC1G07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

Commit message: ready to production
Parts:
- C11, C15, C16, C18, C21, C22, C24, C25: JLCPCB (none) -> C1525; LCSC (none) -> C1525
- C12, C14, C17, C23: JLCPCB (none) -> C15849
- C13: JLCPCB (none) -> C5672
- C19, C20: JLCPCB (none) -> C19702
- C26, C27, C28, C29, C30, C31, C32, C33: JLCPCB (none) -> C15195; LCSC (none) -> C15195
- D11, D12, D13: JLCPCB (none) -> C72041
- D14: JLCPCB (none) -> C72043
- D15, D19, D20: JLCPCB (none) -> C8598
- D16: JLCPCB (none) -> C2286
- D17: JLCPCB (none) -> C2290
- D18: JLCPCB (none) -> C72038
- FB11, FB12: JLCPCB (none) -> C139168
- J11, J12: JLCPCB (none) -> C144395
- J13, J18, J19: JLCPCB (none) -> C144397
- J14: JLCPCB (none) -> C2898761
- R11, R12, R14, R15, R16, R17, R18, R19, R20, R21, R31: JLCPCB (none) -> C25900; LCSC (none) -> C25900
- R13, R23, R24, R25, R26, R27, R28, R29, R30: JLCPCB (none) -> C517529; LCSC (none) -> C517529
- R22: JLCPCB (none) -> C25917; LCSC (none) -> C25917
- R32, R33, R34, R35, R36, R37, R38, R39: JLCPCB (none) -> C11702; LCSC (none) -> C11702
- U11: JLCPCB (none) -> C529338
- U12, U14: JLCPCB (none) -> C5124976
- U13: JLCPCB (none) -> C5148688
- U15: JLCPCB (none) -> C89855
- U16, U17: JLCPCB (none) -> C2836319
